File: grip/pcb/grip/grip.sch (KiCad schematic (older format))
At the start: 4 parts, among them U1 MAN71A, U2 MAN71A

Commit message: added 7 seg footprint, starting layout
Parts:
- R1: footprint (none) -> Resistor_THT:R_Axial_DIN0207_L6.3mm_D2.5mm_P10.16mm_Horizontal
- U1, U2: footprint Display_7Segment:HDSP-7401 -> grip:CAI3191AH
Changed lines of the file:
@@
 F 0 "U1" H 9100 6267 50  0000 C CNN
 F 1 "MAN71A" H 9100 6176 50  0000 C CNN
-F 2 "Display_7Segment:HDSP-7401" H 8600 4900 50  0001 L CNN
+F 2 "grip:CAI3191AH" H 8600 4900 50  0001 L CNN
 F 3 "https://www.digchip.com/datasheets/parts/datasheet/161/MAN3640A-pdf.php" H 9110 5940 50  0001 L CNN
 	1    9100 5600
@@
 F 0 "U2" H 7550 6267 50  0000 C CNN
 F 1 "MAN71A" H 7550 6176 50  0000 C CNN
-F 2 "Display_7Segment:HDSP-7401" H 7050 4900 50  0001 L CNN
+F 2 "grip:CAI3191AH" H 7050 4900 50  0001 L CNN
 F 3 "https://www.digchip.com/datasheets/parts/datasheet/161/MAN3640A-pdf.php" H 7560 5940 50  0001 L CNN
 	1    7550 5600
@@
 U 1 1 5DB6812A
 P 4900 5600
-F 0 "A1" H 4100 6650 50  0000 C CNN
-F 1 "Arduino_Nano_v2.x" H 4150 6500 50  0000 C CNN
+F 0 "A1" H 4900 6800 50  0000 C CNN
+F 1 "Arduino_Nano_v2.x" H 4900 6700 50  0000 C CNN
 F 2 "Module:Arduino_Nano" H 5050 4650 50  0001 L CNN
 F 3 "https://www.arduino.cc/en/uploads/Main/ArduinoNanoManual23.pdf" H 4900 4600 50  0001 C CNN
@@
 $EndComp
 $Comp
-L power:GND #PWR?
+L power:GND #PWR0101
 U 1 1 5DB753D4
 P 7850 6000
-F 0 "#PWR?" H 7850 5750 50  0001 C CNN
+F 0 "#PWR0101" H 7850 5750 50  0001 C CNN
 F 1 "GND" H 7855 5827 50  0000 C CNN
 F 2 "" H 7850 6000 50  0001 C CNN
@@
 $EndComp
 $Comp
-L power:GND #PWR?
+L power:GND #PWR0102
 U 1 1 5DB76090
 P 4900 6600
-F 0 "#PWR?" H 4900 6350 50  0001 C CNN
+F 0 "#PWR0102" H 4900 6350 50  0001 C CNN
 F 1 "GND" H 4905 6427 50  0000 C CNN
 F 2 "" H 4900 6600 50  0001 C CNN
@@
 $EndComp
 $Comp
-L power:GND #PWR?
+L power:GND #PWR0103
 U 1 1 5DB76900
 P 9400 6000
-F 0 "#PWR?" H 9400 5750 50  0001 C CNN
+F 0 "#PWR0103" H 9400 5750 50  0001 C CNN
 F 1 "GND" H 9405 5827 50  0000 C CNN
 F 2 "" H 9400 6000 50  0001 C CNN
@@
 F 0 "R1" H 5970 5996 50  0000 L CNN
 F 1 "1k" H 5970 5905 50  0000 L CNN
-F 2 "" V 5830 5950 50  0001 C CNN
+F 2 "Resistor_THT:R_Axial_DIN0207_L6.3mm_D2.5mm_P10.16mm_Horizontal" V 5830 5950 50  0001 C CNN
 F 3 "~" H 5900 5950 50  0001 C CNN
 	1    5900 5950
@@
 $EndComp
 $Comp
-L power:GND #PWR?
+L power:GND #PWR0104
 U 1 1 5DB67B47
 P 5900 6100
-F 0 "#PWR?" H 5900 5850 50  0001 C CNN
+F 0 "#PWR0104" H 5900 5850 50  0001 C CNN
 F 1 "GND" H 5905 5927 50  0000 C CNN
 F 2 "" H 5900 6100 50  0001 C CNN
